File: eagle/6809.brd (EAGLE design)
At the start: 151.1 x 101.3 mm, 62 parts, among them CN1 2.1MMJACKTHM, IC1 74HC138N, IC2 74HC139N, IC3 74HC541N, IC4 74HC541N, IC5 74HC245N, IC6 74HC00N, IC7 7805TV, T1 PN2222

Commit message: [eagle] some work on a rev 2
Parts:
- removed DE9: COM1, con-subd:F09HP
- removed RX, TX: TPTP10R, testpad:TP10R
- added COM: (no value), con-subd:M09HP
- added JP3: (no value), jumper:JP2
- SV2: device con-lstb:MA04-2 -> con-lstb:MA05-2
- moved IC7 34.3 mm to (14.0, 71.8), turned to 90 degrees
- moved IC3 33.1 mm to (27.3, 15.2)
- moved C17 33.0 mm to (19.1, 29.8), turned to 180 degrees
- moved IC5 32.8 mm to (40.0, 15.2)
- moved TP1 32.6 mm to (8.89, 67.9)
- moved C12 30.5 mm to (20.3, 80.6)
- moved C11 27.0 mm to (22.9, 62.9), turned to 270 degrees
- moved IC4 25.9 mm to (27.3, 43.2)
- moved C7 16.0 mm to (16.5, 61.0)
- moved JP1 14.5 mm to (29.8, 79.4), turned to 270 degrees
- moved TP2 14.0 mm to (9.53, 3.81)
- moved IC6 13.3 mm to (32.4, 66.7)
- moved C2 13.1 mm to (44.7, 33.7), turned to 0 degrees
- moved JP2 12.0 mm to (135.9, 14.6)
- moved TP7 11.5 mm to (70.5, 60.3)
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Connections:
- removed net N$30: IC5.2, SV1.2
- removed net N$31: IC5.3, SV1.4
- removed net N$32: IC5.4, SV1.6
- removed net N$33: IC5.5, SV1.8
- removed net N$34: IC5.6, SV1.10
- removed net N$35: IC5.7, SV1.12
- removed net N$36: IC5.8, SV1.14
- removed net N$37: IC5.9, SV1.16
- new net D0_EXT: IC5.2, SV1.26
- new net D1_EXT: IC5.3, SV1.28
- new net D2_EXT: IC5.4, SV1.30
- new net D3_EXT: IC5.5, SV1.32
- new net D4_EXT: IC5.6, SV1.34
- new net D5_EXT: IC5.7, SV1.36
- new net D6_EXT: IC5.8, SV1.38
- new net D7_EXT: IC5.9, SV1.40
- new net N$24: COM.6, SV2.10
- net !EXTIOSEL0: now also SV1.4; no longer SV1.32
- net !EXTIOSEL1: now also SV1.6; no longer SV1.34
- net !EXTIOSEL2: now also SV1.8; no longer SV1.36
- net !EXTIOSEL3: now also SV1.10; no longer SV1.38
- net !FIRQ: now also SV1.14; no longer SV1.20
- net !IRQ: now also SV1.12; no longer SV1.18
- net !RD: now also IC4.8; no longer IC4.3
- net !RD!_EXT: now also IC4.12, SV1.5; no longer IC4.17, SV1.29
- net !WR: now also IC4.7; no longer IC4.4
- net !WR!_EXT: now also IC4.13, SV1.7; no longer IC4.16, SV1.27
- net A0: now also IC4.6; no longer IC3.9
- net A0_EXT: now also IC4.14, SV1.15; no longer IC3.11, SV1.1
- net A1: now also IC4.5; no longer IC3.8
- net A10: now also IC3.4; no longer IC4.7
- net A10_EXT: now also IC3.16, SV1.35; no longer IC4.13, SV1.21
- net A11: now also IC3.3; no longer IC4.6
- net A11_EXT: now also IC3.17, SV1.37; no longer IC4.14, SV1.23
- net A12: now also IC3.2; no longer IC4.5
- net A12_EXT: now also IC3.18, SV1.39; no longer IC4.15, SV1.25
- net A1_EXT: now also IC4.15, SV1.17; no longer IC3.12, SV1.3
- net A2: now also IC4.4; no longer IC3.7
- net A2_EXT: now also IC4.16, SV1.19; no longer IC3.13, SV1.5
- net A3: now also IC4.3; no longer IC3.6
- net A3_EXT: now also IC4.17, SV1.21; no longer IC3.14, SV1.7
- net A4: now also IC4.2; no longer IC3.5
- net A4_EXT: now also IC4.18, SV1.23; no longer IC3.15, SV1.9
- net A5: now also IC3.9; no longer IC3.4
- net A5_EXT: now also IC3.11, SV1.25; no longer IC3.16, SV1.11
- net A6: now also IC3.8; no longer IC3.3
- net A6_EXT: now also IC3.12, SV1.27; no longer IC3.17, SV1.13
- net A7: now also IC3.7; no longer IC3.2
- net A7_EXT: now also IC3.13, SV1.29; no longer IC3.18, SV1.15
- net A8: now also IC3.6; no longer IC4.9
- net A8_EXT: now also IC3.14, SV1.31; no longer IC4.11, SV1.17
- net A9: now also IC3.5; no longer IC4.8
- net A9_EXT: now also IC3.15, SV1.33; no longer IC4.12, SV1.19
- net CTS: now also SV2.6; no longer SV2.2
- net E: now also IC4.9; no longer IC4.2
- net E_EXT: now also IC4.11, SV1.3; no longer IC4.18, SV1.31
- net GND: now also COM.5, JP3.1, SV1.2; no longer DE9.5, DE9.G1, DE9.G2, SV1.40
- net N$11: now also JP3.3; no longer RX.TP
- net N$16: now also COM.2, SV2.1; no longer DE9.2, SV2.7
- net N$17: now also COM.8; no longer DE9.3
- net N$18: now also COM.7, SV2.7; no longer DE9.7, SV2.3
- net N$20: now also COM.3, SV2.3; no longer DE9.8, SV2.1
- net N$6: now also JP3.2; no longer TX.TP
- net N$8: now also COM.4, SV2.9; no longer DE9.4, DE9.6
- net RTS: now also SV2.8; no longer SV2.4
- net RXD: now also SV2.2; no longer SV2.8
- net TXD: now also SV2.4; no longer SV2.6
- net VCC: now also SV1.1; no longer SV1.39
Routing:
- net !EXTIOSEL0: track 113.6 -> 47.8 mm
- net !EXTIOSEL2: track 106.8 -> 45.2 mm, vias 2 -> 0
- net !RD: track 236.3 -> 180.3 mm, vias 4 -> 3
- net E: track 133.0 -> 77.9 mm
- net !EXTIOSEL3: track 105.0 -> 50.4 mm
- net !WR: track 223.8 -> 170.6 mm, vias 6 -> 5
- net !EXTIOSEL1: track 95.6 -> 45.2 mm, vias 3 -> 0
- net !EXTIOSEL: track 9.83 -> 49.4 mm, vias 0 -> 1
- net D0: track 144.0 -> 105.6 mm, vias 3 -> 2
- net D1: track 145.1 -> 106.9 mm
- net A6: track 148.3 -> 110.4 mm, vias 4 -> 2
- net A2: track 186.2 -> 148.8 mm, vias 3 -> 1
- net A3: track 146.0 -> 109.2 mm, vias 1 -> 0
- net A5: track 143.8 -> 107.1 mm, vias 2 -> 0
- net A7: track 147.3 -> 110.8 mm, vias 4 -> 2
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Other:
- board size 151.1 x 101.3 mm -> 139.7 x 101.3 mm
- board text added: "!WE! Enable"
- board text added: "6809 Mainboard Rev 1.99"
- board text added: "GND"
- board text added: "RX"
- board text added: "TX"
- board text added: "VCC"
- board text removed: "6809 Mainboard Rev 1"
