File: eagle/6809.sch (EAGLE design)
At the start: 62 parts, among them CN1 2.1MMJACKTHM, IC1 74HC138N, IC2 74HC139N, IC3 74HC541N, IC4 74HC541N, IC5 74HC245N, IC6 74HC00N, IC7 7805TV, T1 PN2222

Commit message: [eagle] some work on a rev 2
Parts:
- removed DE9: COM1, con-subd:F09HP
- removed RX, TX: TPTP10R, testpad:TPTP10R
- added COM: (no value), con-subd:M09HP
- added JP3: (no value), jumper:JP2E
- SV2: device con-lstb:MA04-2 -> con-lstb:MA05-2
Connections:
- removed net N$30: IC5A.A1, SV1.2
- removed net N$31: IC5A.A2, SV1.4
- removed net N$32: IC5A.A3, SV1.6
- removed net N$33: IC5A.A4, SV1.8
- removed net N$34: IC5A.A5, SV1.10
- removed net N$35: IC5A.A6, SV1.12
- removed net N$36: IC5A.A7, SV1.14
- removed net N$37: IC5A.A8, SV1.16
- new net D0_EXT: IC5A.A1, SV1.26
- new net D1_EXT: IC5A.A2, SV1.28
- new net D2_EXT: IC5A.A3, SV1.30
- new net D3_EXT: IC5A.A4, SV1.32
- new net D4_EXT: IC5A.A5, SV1.34
- new net D5_EXT: IC5A.A6, SV1.36
- new net D6_EXT: IC5A.A7, SV1.38
- new net D7_EXT: IC5A.A8, SV1.40
- new net N$24: COM.6, SV2.10
- net !EXTIOSEL0: now also SV1.4; no longer SV1.32
- net !EXTIOSEL1: now also SV1.6; no longer SV1.34
- net !EXTIOSEL2: now also SV1.8; no longer SV1.36
- net !EXTIOSEL3: now also SV1.10; no longer SV1.38
- net !FIRQ: now also SV1.14; no longer SV1.20
- net !IRQ: now also SV1.12; no longer SV1.18
- net !RD: now also IC4A.A7; no longer IC4A.A2
- net !RD!_EXT: now also IC4A.Y7, SV1.5; no longer IC4A.Y2, SV1.29
- net !WR: now also IC4A.A6; no longer IC4A.A3
- net !WR!_EXT: now also IC4A.Y6, SV1.7; no longer IC4A.Y3, SV1.27
- net A0: now also IC4A.A5; no longer IC3A.A8
- net A0_EXT: now also IC4A.Y5, SV1.15; no longer IC3A.Y8, SV1.1
- net A1: now also IC4A.A4; no longer IC3A.A7
- net A10: now also IC3A.A3; no longer IC4A.A6
- net A10_EXT: now also IC3A.Y3, SV1.35; no longer IC4A.Y6, SV1.21
- net A11: now also IC3A.A2; no longer IC4A.A5
- net A11_EXT: now also IC3A.Y2, SV1.37; no longer IC4A.Y5, SV1.23
- net A12: now also IC3A.A1; no longer IC4A.A4
- net A12_EXT: now also IC3A.Y1, SV1.39; no longer IC4A.Y4, SV1.25
- net A1_EXT: now also IC4A.Y4, SV1.17; no longer IC3A.Y7, SV1.3
- net A2: now also IC4A.A3; no longer IC3A.A6
- net A2_EXT: now also IC4A.Y3, SV1.19; no longer IC3A.Y6, SV1.5
- net A3: now also IC4A.A2; no longer IC3A.A5
- net A3_EXT: now also IC4A.Y2, SV1.21; no longer IC3A.Y5, SV1.7
- net A4: now also IC4A.A1; no longer IC3A.A4
- net A4_EXT: now also IC4A.Y1, SV1.23; no longer IC3A.Y4, SV1.9
- net A5: now also IC3A.A8; no longer IC3A.A3
- net A5_EXT: now also IC3A.Y8, SV1.25; no longer IC3A.Y3, SV1.11
- net A6: now also IC3A.A7; no longer IC3A.A2
- net A6_EXT: now also IC3A.Y7, SV1.27; no longer IC3A.Y2, SV1.13
- net A7: now also IC3A.A6; no longer IC3A.A1
- net A7_EXT: now also IC3A.Y6, SV1.29; no longer IC3A.Y1, SV1.15
- net A8: now also IC3A.A5; no longer IC4A.A8
- net A8_EXT: now also IC3A.Y5, SV1.31; no longer IC4A.Y8, SV1.17
- net A9: now also IC3A.A4; no longer IC4A.A7
- net A9_EXT: now also IC3A.Y4, SV1.33; no longer IC4A.Y7, SV1.19
- net CTS: now also SV2.6; no longer SV2.2
- net E: now also IC4A.A8; no longer IC4A.A1
- net E_EXT: now also IC4A.Y8, SV1.3; no longer IC4A.Y1, SV1.31
- net GND: now also COM.5, JP3.1, SV1.2; no longer DE9.5, DE9.G1, DE9.G2, SV1.40
- net N$11: now also JP3.3; no longer RX.TP
- net N$16: now also COM.2, SV2.1; no longer DE9.2, SV2.7
- net N$17: now also COM.8; no longer DE9.3
- net N$18: now also COM.7, SV2.7; no longer DE9.7, SV2.3
- net N$20: now also COM.3, SV2.3; no longer DE9.8, SV2.1
- net N$6: now also JP3.2; no longer TX.TP
- net N$8: now also COM.4, SV2.9; no longer DE9.4, DE9.6
- net RTS: now also SV2.8; no longer SV2.4
- net RXD: now also SV2.2; no longer SV2.8
- net TXD: now also SV2.4; no longer SV2.6
- net VCC: now also SV1.1; no longer SV1.39
Other:
- note added: "6809 Mainboard Rev 1.99 (C) 2014, Travis Geiselbrecht geist@foobox.com"
- moved on the sheet: IC5, IC5P, SV1
